Commit message: Phase 2: simulated stereo cameras, rectification, and depth
- robo_description/urdf/robo.gazebo.xacro: <sensor type="camera"> blocks on
  camera_left_link / camera_right_link, 1280x720, 1.086 rad (62.2 deg) hFOV,
  30 Hz, matching camera_update_rate on both so gz-sim's deterministic
  sim-stepped Sensors system produces identical timestamps. optical_frame_id
  set to the REP-103 optical links from Phase 0 so message frame_ids match
  what argus_stereo_node will publish on real hardware.
- robo_sim/config/bridge.yaml: extended with the four stereo topics
  (/stereo/{left,right}/{image_raw,camera_info}), mapped from gz-sim's
  default scoped sensor topic names to the exact Section 3 contract names.
- robo_bringup/launch/common.launch.py: adds a composable node container
  with isaac_ros_image_proc::RectifyNode (x2) and isaac_ros_stereo_image_proc
  Disparity/PointCloud nodes, producing /stereo/{left,right}/image_rect +
  camera_info_rect, /stereo/disparity, and /stereo/points2 (throttled to
  10 Hz).

BLOCKED, flagging explicitly per instructions: isaac_ros_image_proc and
isaac_ros_stereo_image_proc are Isaac ROS / JetPack 6 packages not
installable on this Windows dev machine, so the Phase 2 gate (RViz showing
/stereo/left/image_rect + /stereo/right/image_rect with matching stamps and
a recognizable /stereo/points2) could not be run or verified here. The nodes
are gated behind the enable_isaac_ros launch arg (default false, logs an
explicit notice when off) so sim.launch.py still runs cleanly without them;
flip enable_isaac_ros:=true on the Jetson where Isaac ROS is installed.

Co-Authored-By: Claude Sonnet 5 <noreply@anthropic.com>

File: ros2_ws/src/robo_description/urdf/robo.gazebo.xacro (robot description, xacro)
@@ -5,5 +5,4 @@
   base xacro loads on the real robot with none of this present and the TF tree stays
   identical between sim and hardware (Section 4/6).
-  Phase 2 adds: stereo camera sensors on camera_left_link / camera_right_link.
 -->
 <robot xmlns:xacro="http://www.ros.org/wiki/xacro">
@@ -33,3 +32,55 @@
     </plugin>
   </gazebo>
+  <!-- Stereo cameras: attached to the X-forward camera_*_link (not the
+       *_optical link) since gz-sim's default camera sensor look direction is
+       the parent frame's local +X, matching our URDF convention. optical_frame_id
+       overrides the published frame_id to the REP-103 optical frame defined in
+       robo.urdf.xacro, so downstream consumers (rectify, VSLAM, stereo_image_proc)
+       see the same frame_id in sim as they will from argus_stereo_node on real
+       hardware. No <topic> override: left as the gz-sim default scoped topic
+       name (.../link/<link>/sensor/<name>/image|camera_info) so it lines up
+       with robo_sim/config/bridge.yaml's gz_topic_name entries.
+       Both sensors share camera_update_rate so gz-sim's deterministic,
+       sim-time-stepped Sensors system ticks them on the same simulation step;
+       there is no additional "sync" plugin needed for that in sim. -->
+  <gazebo reference="camera_left_link">
+    <sensor name="left_camera" type="camera">
+      <always_on>true</always_on>
+      <update_rate>${camera_update_rate}</update_rate>
+      <visualize>true</visualize>
+      <optical_frame_id>camera_left_optical</optical_frame_id>
+      <camera>
+        <horizontal_fov>${camera_hfov}</horizontal_fov>
+        <image>
+          <width>${camera_width_px}</width>
+          <height>${camera_height_px}</height>
+          <format>R8G8B8</format>
+        </image>
+        <clip>
+          <near>0.05</near>
+          <far>30.0</far>
+        </clip>
+      </camera>
+    </sensor>
+  </gazebo>
+  <gazebo reference="camera_right_link">
+    <sensor name="right_camera" type="camera">
+      <always_on>true</always_on>
+      <update_rate>${camera_update_rate}</update_rate>
+      <visualize>true</visualize>
+      <optical_frame_id>camera_right_optical</optical_frame_id>
+      <camera>
+        <horizontal_fov>${camera_hfov}</horizontal_fov>
+        <image>
+          <width>${camera_width_px}</width>
+          <height>${camera_height_px}</height>
+          <format>R8G8B8</format>
+        </image>
+        <clip>
+          <near>0.05</near>
+          <far>30.0</far>
+        </clip>
+      </camera>
+    </sensor>
+  </gazebo>
 </robot>
